File: pcb_for_cnc_for_pcb/board/board.kicad_pcb (KiCad board)
At the start: 2 copper layers, 27 parts

Commit message: admin
Parts:
- moved Ymin1 81.5 mm to (206.5, 100.1), turned to 90 degrees
- moved D1 76.9 mm to (205.6, 87.3), turned to 90 degrees
- moved Zmin1 76.5 mm to (206.5, 61.6), turned to 90 degrees
- moved Zmax1 74.0 mm to (206.5, 73.6), turned to 90 degrees
- moved C3 66.8 mm to (215.8, 95.3), turned to -90 degrees
- moved C5 66.4 mm to (215.8, 56.8), turned to -90 degrees
- moved Xmax1 66.0 mm to (224.0, 107.0), turned to 90 degrees
- moved C6 61.6 mm to (215.8, 68.8), turned to -90 degrees
- moved R1 61.3 mm to (215.6, 80.0), turned to 180 degrees
- moved 5Vacces1 58.6 mm to (219.0, 87.5), turned to 90 degrees
- moved C2 52.0 mm to (233.3, 102.2), turned to -90 degrees
- moved Ymax1 50.5 mm to (242.5, 107.0), turned to 90 degrees
- moved A1 40.0 mm to (238.1, 95.0), turned to 180 degrees
- moved C4 39.8 mm to (251.8, 102.2), turned to -90 degrees
- moved Pwm1 35.4 mm to (244.0, 55.5), turned to 90 degrees
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Routing:
- net (no net): track 0.00 -> 30.4 mm
- net Net-(D1-K): track 41.3 -> 48.6 mm
- net Net-(A1-SDA/A4): track 75.0 -> 72.9 mm
- net Net-(A1-D10/CS): track 28.9 -> 27.5 mm
- net Net-(A1-D2): track 30.5 -> 29.5 mm
- net Net-(A1-D11/COPI): track 8.97 -> 9.56 mm

Commit message: webdisajn
Parts:
- moved Ymin1 2.50 mm to (209.0, 100.1)
- moved R1 2.00 mm to (217.6, 80.0)
- moved Zmax1 2.00 mm to (208.5, 73.6)
- moved Zmin1 2.00 mm to (208.5, 61.6)
- moved D1 1.96 mm to (207.5, 87.3)
Routing:
- net (no net): track 30.4 -> 0.00 mm
- net Net-(A1-A3): track 42.9 -> 38.7 mm
- net Net-(A1-SCL/A5): track 7.37 -> 5.37 mm
- net Net-(A1-A1): track 18.2 -> 16.2 mm
- net Net-(A1-A0): track 24.7 -> 22.7 mm
- net Net-(A1-SDA/A4): track 72.9 -> 71.4 mm
- net Net-(D1-K): track 48.6 -> 47.6 mm
- net Net-(A1-VUSB/5V): track 4.40 -> 4.90 mm
Other:
- board text removed: "Cnc control panel"
